File: boards/prox-sense-single-mtch105-v0.1/prox-sense-single-mtch105-omni-v0.1-19.05mm-handsolder/prox-sense-single-mtch105-omni-v0.1-19.05mm-handsolder.kicad_pcb (KiCad board)
At the start: 2 copper layers, 24.7 x 48.6 mm, 11 parts, among them J1 Conn_01x04_Male, U1 MTCH105, U2 prox-sense-cap

Commit message: gerber zip, omni guard on one side, no vias
Parts:
- U2: moved to F.Cu
- turned U2 to 0 degrees
Routing:
- net SENSE0: vias 1 -> 0
